File: Team2 Sch with Power and Battery.kicad_sch (KiCad schematic)
At the start: 76 parts, among them J1 Conn_01x05, J10 Conn_01x03_MountingPin, J11 Conn_01x03_MountingPin, J12 Conn_01x03_MountingPin, J13 Conn_01x03_MountingPin, J14 Conn_01x03_MountingPin, J15 Conn_01x03_Pin, J16 Conn_01x08_Pin, J17 XT60-M, J18 XT60-M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

Commit message: Latest version Battery 8-29
Parts:
- added R31: 2k Ohm, symbol Device:R_Small_US
Connections:
- net +12V: now also SW2.2, R31.1
- net at D1.2 (A): now also R31.2; no longer SW2.2
Other:
- moved on the sheet: D1
Changed lines of the file:
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@@
 	)
 	(junction
-		(at 464.82 59.69)
+		(at 276.86 35.56)
 		(diameter 0)
 		(color 0 0 0 0)
 	)
 	(junction
-		(at 276.86 35.56)
+		(at 449.58 59.69)
 		(diameter 0)
 		(color 0 0 0 0)
@@
 	)
 	(junction
+		(at 468.63 59.69)
+		(diameter 0)
+		(color 0 0 0 0)
+	)
+	(junction
 		(at 187.96 246.38)
 		(diameter 0)
@@
 	)
 	(junction
+		(at 462.28 59.69)
+		(diameter 0)
+		(color 0 0 0 0)
+	)
+	(junction
 		(at 415.29 59.69)
 		(diameter 0)
@@
 	)
 	(junction
-		(at 464.82 53.34)
+		(at 468.63 53.34)
 		(diameter 0)
 		(color 0 0 0 0)
@@
 	(wire
 		(pts
-			(xy 447.04 59.69) (xy 450.85 59.69)
-		)
-		(stroke
-			(width 0)
-			(type default)
-		)
-	)
-	(wire
-		(pts
 			(xy 446.405 154.305) (xy 446.405 155.575)
 		)
@@
 	(wire
 		(pts
-			(xy 464.82 59.69) (xy 464.82 53.34)
+			(xy 468.63 53.34) (xy 468.63 59.69)
 		)
 		(stroke
@@
 	(wire
 		(pts
+			(xy 462.28 59.69) (xy 468.63 59.69)
+		)
+		(stroke
+			(width 0)
+			(type default)
+		)
+	)
+	(wire
+		(pts
 			(xy 415.29 72.39) (xy 415.29 74.93)
 		)
@@
 	(wire
 		(pts
-			(xy 464.82 59.69) (xy 464.82 69.85)
-		)
-		(stroke
-			(width 0)
-			(type default)
-		)
-	)
-	(wire
-		(pts
 			(xy 287.02 276.86) (xy 287.02 281.94)
 		)
@@
 	(wire
 		(pts
+			(xy 449.58 55.88) (xy 449.58 59.69)
+		)
+		(stroke
+			(width 0)
+			(type default)
+		)
+	)
+	(wire
+		(pts
 			(xy 288.29 147.32) (xy 292.1 147.32)
 		)
@@
 	(wire
 		(pts
+			(xy 462.28 55.88) (xy 462.28 59.69)
+		)
+		(stroke
+			(width 0)
+			(type default)
+		)
+	)
+	(wire
+		(pts
 			(xy 288.29 152.4) (xy 283.21 152.4)
 		)
@@
 	(wire
 		(pts
+			(xy 468.63 59.69) (xy 468.63 69.85)
+		)
+		(stroke
+			(width 0)
+			(type default)
+		)
+	)
+	(wire
+		(pts
+			(xy 447.04 59.69) (xy 449.58 59.69)
+		)
+		(stroke
+			(width 0)
+			(type default)
+		)
+	)
+	(wire
+		(pts
 			(xy 287.02 281.94) (xy 281.94 281.94)
 		)
@@
 	(wire
 		(pts
-			(xy 464.82 45.72) (xy 464.82 53.34)
+			(xy 468.63 45.72) (xy 468.63 53.34)
 		)
 		(stroke
@@
 	(wire
 		(pts
-			(xy 458.47 59.69) (xy 464.82 59.69)
+			(xy 415.29 59.69) (xy 415.29 64.77)
 		)
 		(stroke
@@
 	(wire
 		(pts
-			(xy 415.29 59.69) (xy 415.29 64.77)
+			(xy 415.29 59.69) (xy 422.91 59.69)
 		)
 		(stroke
@@
 	(wire
 		(pts
-			(xy 415.29 59.69) (xy 422.91 59.69)
+			(xy 449.58 59.69) (xy 462.28 59.69)
 		)
 		(stroke
@@
 	(wire
 		(pts
-			(xy 464.82 53.34) (xy 467.36 53.34)
+			(xy 468.63 53.34) (xy 471.17 53.34)
 		)
 		(stroke
@@
 	(text "voltage regulator\n"
 		(exclude_from_sim no)
-		(at 448.31 63.5 0)
+		(at 460.756 62.23 0)
 		(effects
 			(font
@@
 	(symbol
 		(lib_id "Device:LED")
-		(at 454.66 59.69 180)
+		(at 458.47 55.88 180)
 		(unit 1)
 		(exclude_from_sim no)
@@
 		(fields_autoplaced yes)
 		(property "Reference" "D1"
-			(at 456.2475 52.07 0)
+			(at 460.0575 48.26 0)
 			(effects
 				(font
@@
 		)
 		(property "Value" "LED"
-			(at 456.2475 54.61 0)
+			(at 460.0575 50.8 0)
 			(effects
 				(font
@@
 		)
 		(property "Footprint" ""
-			(at 454.66 59.69 0)
+			(at 458.47 55.88 0)
 			(effects
 				(font
@@
 		)
 		(property "Datasheet" "~"
-			(at 454.66 59.69 0)
+			(at 458.47 55.88 0)
 			(effects
 				(font
@@
 		)
 		(property "Description" "Light emitting diode"
-			(at 454.66 59.69 0)
+			(at 458.47 55.88 0)
 			(effects
 				(font
@@
 	(symbol
 		(lib_id "power:+5V")
-		(at 464.82 45.72 0)
+		(at 468.63 45.72 0)
 		(unit 1)
 		(exclude_from_sim no)
@@
 		(fields_autoplaced yes)
 		(property "Reference" "#PWR058"
-			(at 464.82 49.53 0)
+			(at 468.63 49.53 0)
 			(effects
 				(font
@@
 		)
 		(property "Value" "+5V"
-			(at 464.82 40.64 0)
+			(at 468.63 40.64 0)
 			(effects
 				(font
@@
 		)
 		(property "Footprint" ""
-			(at 464.82 45.72 0)
+			(at 468.63 45.72 0)
 			(effects
 				(font
@@
 		)
 		(property "Datasheet" ""
-			(at 464.82 45.72 0)
+			(at 468.63 45.72 0)
 			(effects
 				(font
@@
 		)
 		(property "Description" "Power symbol creates a global label with name \"+5V\""
-			(at 464.82 45.72 0)
+			(at 468.63 45.72 0)
 			(effects
 				(font
@@
 	(symbol
 		(lib_id "power:+12V")
-		(at 464.82 69.85 180)
+		(at 468.63 69.85 180)
 		(unit 1)
 		(exclude_from_sim no)
@@
 		(fields_autoplaced yes)
 		(property "Reference" "#PWR059"
-			(at 464.82 66.04 0)
+			(at 468.63 66.04 0)
 			(effects
 				(font
@@
 		)
 		(property "Value" "+12V"
-			(at 464.82 74.93 0)
+			(at 468.63 74.93 0)
 			(effects
 				(font
@@
 		)
 		(property "Footprint" ""
-			(at 464.82 69.85 0)
+			(at 468.63 69.85 0)
 			(effects
 				(font
@@
 		)
 		(property "Datasheet" ""
-			(at 464.82 69.85 0)
+			(at 468.63 69.85 0)
 			(effects
 				(font
@@
 		)
 		(property "Description" "Power symbol creates a global label with name \"+12V\""
-			(at 464.82 69.85 0)
+			(at 468.63 69.85 0)
 			(effects
 				(font
@@
 					(unit 1)
 				)
+			)
+		)
+	)
+	(symbol
+		(lib_id "Device:R_Small_US")
+		(at 452.12 55.88 90)
+		(unit 1)
+		(exclude_from_sim no)
+		(in_bom yes)
+		(on_board yes)
+		(dnp no)
+		(fields_autoplaced yes)
+		(property "Reference" "R31"
+			(at 452.12 49.53 90)
+			(effects
+				(font
+					(size 1.27 1.27)
+				)
+			)
+		)
+		(property "Value" "2k Ohm"
+			(at 452.12 52.07 90)
+			(effects
+				(font
+					(size 1.27 1.27)
+				)
+			)
+		)
+		(property "Footprint" ""
+			(at 452.12 55.88 0)
+			(effects
+				(font
+					(size 1.27 1.27)
+				)
+				(hide yes)
+			)
+		)
+		(property "Datasheet" "~"
+			(at 452.12 55.88 0)
+			(effects
+				(font
+					(size 1.27 1.27)
+				)
+				(hide yes)
+			)
+		)
+		(property "Description" "Resistor, small US symbol"
+			(at 452.12 55.88 0)
+			(effects
+				(font
+					(size 1.27 1.27)
+				)
+				(hide yes)
+			)
+		)
+		(pin "2"
+		)
+		(pin "1"
+		)
+		(instances
+			(project ""
+				(path "/113d5a4f-8af6-4d26-a733-e9d3dd2d040f"
+					(reference "R31")
+					(unit 1)
+				)
