File: Team2.kicad_sch (KiCad schematic)
At the start: 71 parts, among them J1 Conn_01x05, J10 Conn_01x03_MountingPin, J11 Conn_01x03_MountingPin, J12 Conn_01x03_MountingPin, J13 Conn_01x03_MountingPin, J14 Conn_01x03_MountingPin, J15 Conn_01x03_Pin, J16 Conn_01x08_Pin, J17 XT60-M, J18 XT60-M, J2 Conn_01x03_MountingPin, J20 Conn_01x05, J3 Conn_01x03_MountingPin, J4 Conn_01x03_MountingPin, J5 Conn_01x03_MountingPin, J6 Conn_01x03_MountingPin, J7 Conn_01x03_MountingPin, J8 Conn_01x03_MountingPin, J9 Conn_01x03_MountingPin, Q1 SQM40P10-40L_GE3, Q2 SQ2318AES-T1_BE3, SW1 SW_SPST, U2 Teensy4.1

Commit message: 8-29-24 8:55
Parts:
- added C18, C19, C20, C21: 100nF, symbol Device:C_Small
- added D1, D10, D11, D12, D13, D2, D3, D4, D5, D6, D7, D8, D9: LED, symbol Device:LED
- added R31, R32, R33, R34, R35, R36, R37, R38, R39, R40, R41, R42, R43: R, symbol Device:R
- added U1: S-1142DA0I-E6T1U, HSOP6-A-PKG_FH006-A-P-SD-2.1_ABL, symbol voltage reg 12v:S-1142DA0I-E6T1U
- added U3: TQL850CSV50_RLG, TQL850CSV50_RLG:SOIC127P600X170-9N, symbol voltage reg. 5v:TQL850CSV50_RLG
Connections:
- net Distance Sensor 1 3.3V: now also R35.1
- net Distance Sensor 2 3.3V: now also R36.1
- net Distance Sensor 3 3.3V: now also R37.1
- net Distance Sensor 4 3.3V: now also R38.1
- net Distance Sensor 5 3.3V: now also R39.1
- net Distance Sensor 6 3.3V: now also R40.1
- net Distance Sensor 7 3.3V: now also R41.1
- net Distance Sensor 8 3.3V: now also R42.1
- net Distance Sensor 9 3.3V: now also R43.1
- net GND: now also C18.2, C19.2, C20.2, C21.2, U1.2 (VSS), U1.5 (VSS), U3.4 (GND), U3.5 (RTH), U3.6 (WDI)
- net GND1: now also D1.1 (K), D10.1 (K), D11.1 (K), D12.1 (K), D13.1 (K), D2.1 (K), D3.1 (K), D4.1 (K), D5.1 (K), D6.1 (K), D7.1 (K), D8.1 (K), D9.1 (K)
- net Line Sensor 1 3.3V: now also R31.1
- net Line Sensor 2 3.3V: now also R32.1
- net Line Sensor 3 3.3V: now also R33.1
- net Line Sensor 4 3.3V: now also R34.1
- new net: D4.2 (A), R34.2
- new net: D9.2 (A), R39.2
- new net: D2.2 (A), R32.2
- new net: D10.2 (A), R40.2
- new net: D3.2 (A), R33.2
- new net: D8.2 (A), R38.2
- new net: D12.2 (A), R42.2
- new net: D7.2 (A), R37.2
- new net: D6.2 (A), R36.2
- new net: D5.2 (A), R35.2
- new net: D1.2 (A), R31.2
- new net: D11.2 (A), R41.2
- new net: D13.2 (A), R43.2
- new net 12v: C19.1, U1.1 (VOUT), U1.3 (ON/OFF)
- new net 44.4v: C18.1, C20.1, U1.6 (VIN), U3.1 (IN), U3.2 (EN)
- new net 5v: C21.1, U3.8 (OUT)
- no-connect marks 3 -> 5
Other:
- note added: "Resistors 31-34 are 40 Ohm"
- note added: "Resistors 35-43 are 3 Ohm"
- note added: "Voltage Regulators"
- moved on the sheet: C15, C16, C17, F1, J17, J18, Q1, Q2, R27, R28, R29, R30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
