File: Team2/Team2.kicad_sch (KiCad schematic)
At the start: 70 parts, among them J1 Conn_01x04_MountingPin, J10 Conn_01x03_MountingPin, J11 Conn_01x03_MountingPin, J12 Conn_01x03_MountingPin, J13 Conn_01x03_MountingPin, J14 Conn_01x03_MountingPin, J15 Conn_01x03_Pin, J16 Conn_01x08_Pin, J17 XT60-M, J18 XT60-M, J2 Conn_01x03_MountingPin, J3 Conn_01x03_MountingPin, J4 Conn_01x03_MountingPin, J5 Conn_01x03_MountingPin, J6 Conn_01x03_MountingPin, J7 Conn_01x03_MountingPin, J8 Conn_01x03_MountingPin, J9 Conn_01x03_MountingPin, Q1 SQM40P10-40L_GE3, Q2 SQ2318AES-T1_BE3, SW1 SW_SPST, U2 Teensy4.1

Commit message: 8-29-24 8:55
Parts:
- removed J1: Conn_01x04_MountingPin, Connector_JST:JST_PH_B4B-PH-SM4-TB_1x04-1MP_P2.00mm_Vertical, symbol Connector_Generic_MountingPin:Conn_01x04_MountingPin
- added C18, C19, C20, C21: 100nF, symbol Device:C_Small
- added D1, D10, D11, D12, D13, D2, D3, D4, D5, D6, D7, D8, D9: LED, symbol Device:LED
- added J1, J20: Conn_01x05, symbol Connector_Generic:Conn_01x05
- added R31, R32, R33, R34, R35, R36, R37, R38, R39, R40, R41, R42, R43: R, symbol Device:R
- added U1: S-1142DA0I-E6T1U, HSOP6-A-PKG_FH006-A-P-SD-2.1_ABL, symbol voltage reg 12v:S-1142DA0I-E6T1U
- added U3: TQL850CSV50_RLG, TQL850CSV50_RLG:SOIC127P600X170-9N, symbol voltage reg. 5v:TQL850CSV50_RLG
Connections:
- net +5V: now also J1.3 (Pin_3), J20.3 (Pin_3)
- net 44.4V: now also J1.5 (Pin_5), J20.5 (Pin_5)
- net Distance Sensor 1 3.3V: now also R35.1
- net Distance Sensor 2 3.3V: now also R36.1
- net Distance Sensor 3 3.3V: now also R37.1
- net Distance Sensor 4 3.3V: now also R38.1
- net Distance Sensor 5 3.3V: now also R39.1
- net Distance Sensor 6 3.3V: now also R40.1
- net Distance Sensor 7 3.3V: now also R41.1
- net Distance Sensor 8 3.3V: now also R42.1
- net Distance Sensor 9 3.3V: now also R43.1
- net GND: now also C18.2, C19.2, C20.2, C21.2, U1.2 (VSS), U1.5 (VSS), U3.4 (GND), U3.5 (RTH), U3.6 (WDI)
- net GND1: now also D1.1 (K), D10.1 (K), D11.1 (K), D12.1 (K), D13.1 (K), D2.1 (K), D3.1 (K), D4.1 (K), D5.1 (K), D6.1 (K), D7.1 (K), D8.1 (K), D9.1 (K), J1.4 (Pin_4), J20.4 (Pin_4)
- net Interupt: now also U2.39 (17_A3_TX4_SDA1)
- net Line Sensor 1 3.3V: now also R31.1
- net Line Sensor 2 3.3V: now also R32.1
- net Line Sensor 3 3.3V: now also R33.1
- net Line Sensor 4 3.3V: now also R34.1
- net SCL: now also U2.41 (19_A5_SCL)
- net SDA: now also U2.40 (18_A4_SDA)
- net PWM MD2: now reaches U2.6 (4_BCLK2)
- net PWM MD2: now also J20.2 (Pin_2)
- net Direction MD: no longer names the net of U2.4 (2_OUT2)
- net PWM MD renamed Direction MD2
- net Direction MD2: now also J20.1 (Pin_1)
- new net: D4.2 (A), R34.2
- new net: D9.2 (A), R39.2
- new net: D2.2 (A), R32.2
- new net: D10.2 (A), R40.2
- new net: D3.2 (A), R33.2
- new net: D8.2 (A), R38.2
- new net: D12.2 (A), R42.2
- new net: D7.2 (A), R37.2
- new net: D6.2 (A), R36.2
- new net: D5.2 (A), R35.2
- new net: D1.2 (A), R31.2
- new net: D11.2 (A), R41.2
- new net: D13.2 (A), R43.2
- new net 12v: C19.1, U1.1 (VOUT), U1.3 (ON/OFF)
- new net 44.4v: C18.1, C20.1, U1.6 (VIN), U3.1 (IN), U3.2 (EN)
- new net 5v: C21.1, U3.8 (OUT)
- new net Direction MD1: J1.1 (Pin_1)
- new net PWM MD1: J1.2 (Pin_2)
- no-connect marks 3 -> 5
Other:
- note added: "IMU"
- note added: "Resistors 31-34 are 40 Ohm"
- note added: "Resistors 35-43 are 3 Ohm"
- note added: "Voltage Regulators"
- note added: "Voltage divider 12V to 3.3V using 3.6kOhms and 9.1kOhms resistors. Not sure how we would keep ground planes sep"
- note removed: "Voltage divider 12V to 3.3V using 3.6kOhms and 9.1kOhms resistors."
- moved on the sheet: C14, C15, C16, C17, F1, J15, J17, J18, Q1, Q2, R27, R28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

Commit message: Use team 2 New
Parts:
- removed C18, C19, C20, C21: 100nF, symbol Device:C_Small
- removed D1, D10, D11, D12, D13, D2, D3, D4, D5, D6, D7, D8, D9: LED, symbol Device:LED
- removed J1, J20: Conn_01x05, symbol Connector_Generic:Conn_01x05
- removed R31, R32, R33, R34, R35, R36, R37, R38, R39, R40, R41, R42, R43: R, symbol Device:R
- removed U1: S-1142DA0I-E6T1U, HSOP6-A-PKG_FH006-A-P-SD-2.1_ABL, symbol voltage reg 12v:S-1142DA0I-E6T1U
- removed U3: TQL850CSV50_RLG, TQL850CSV50_RLG:SOIC127P600X170-9N, symbol voltage reg. 5v:TQL850CSV50_RLG
- added J1: Conn_01x04_MountingPin, Connector_JST:JST_PH_B4B-PH-SM4-TB_1x04-1MP_P2.00mm_Vertical, symbol Connector_Generic_MountingPin:Conn_01x04_MountingPin
Connections:
- net +5V: now also J1.3 (Pin_3)
- net GND1: now also J1.4 (Pin_4)
- net Interupt: no longer U2.39 (17_A3_TX4_SDA1)
- net SCL: no longer U2.41 (19_A5_SCL)
- net SDA: no longer U2.40 (18_A4_SDA)
- net Direction MD: now reaches U2.4 (2_OUT2)
- net Direction MD: now also J1.1 (Pin_1)
- net Direction MD2 renamed PWM MD
- net PWM MD: now also J1.2 (Pin_2)
- net PWM MD2: no longer names the net of U2.6 (4_BCLK2)
- no-connect marks 5 -> 3
Other:
- note added: "C1-14 are .1µF"
- note added: "Voltage divider 12V to 3.3V using 3.6kOhms and 9.1kOhms resistors."
- note removed: "C1-13 are .1µF"
- note removed: "IMU"
- note removed: "Resistors 31-34 are 40 Ohm"
- note removed: "Resistors 35-43 are 3 Ohm"
- note removed: "Voltage Regulators"
- note removed: "Voltage divider 12V to 3.3V using 3.6kOhms and 9.1kOhms resistors. Not sure how we would keep ground planes sep"
- moved on the sheet: C14, C15, C16, C17, F1, J15, J17, J18, Q1, Q2, R27, R28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
