File: Team2/_autosave-Team2-New.kicad_sch (KiCad schematic)
At the start: 109 parts, among them J1 Conn_01x05, J10 Conn_01x03_MountingPin, J11 Conn_01x03_MountingPin, J12 Conn_01x03_MountingPin, J13 Conn_01x03_MountingPin, J14 Conn_01x03_MountingPin, J15 Conn_01x03_Pin, J16 Conn_01x08_Pin, J17 XT60-M, J18 XT60-M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

Commit message: updates 7/1
Parts:
- added D15, D16: LED, symbol Device:LED
- added R45, R46: R, symbol Device:R
Connections:
- net 12v: now also R45.1
- net 5v: now also R46.1
- net GND1: now also D15.1 (K), D16.1 (K)
- new net: D15.2 (A), R45.2
- new net: D16.2 (A), R46.2
Other:
- moved on the sheet: D14, F2, F3, J19, R44, SW2
