File: Team2/Team2-New.kicad_sch (KiCad schematic)
At the start: 109 parts, among them J1 Conn_01x05, J10 Conn_01x03_MountingPin, J11 Conn_01x03_MountingPin, J12 Conn_01x03_MountingPin, J13 Conn_01x03_MountingPin, J14 Conn_01x03_MountingPin, J15 Conn_01x03_Pin, J16 Conn_01x08_Pin, J17 XT60-M, J18 XT60-M, J19 Battery Connector, J2 Conn_01x03_MountingPin, J20 Conn_01x05, J3 Conn_01x03_MountingPin, J4 Conn_01x03_MountingPin, J5 Conn_01x03_MountingPin, J6 Conn_01x03_MountingPin, J7 Conn_01x03_MountingPin, J8 Conn_01x03_MountingPin, J9 Conn_01x03_MountingPin, Q1 SQM40P10-40L_GE3, Q2 SQ2318AES-T1_BE3, SW1 SW_SPST, SW2 SW_DIP_x01, U1 S-1142DA0I-E6T1U, U2 Teensy4.1, U3 TQL850CSV50_RLG

Commit message: ok
Parts:
- added C22: C, symbol Device:C
- added D15, D16: LED, symbol Device:LED
- added R45, R46: R, symbol Device:R
Connections:
- net +12V: now also C22.1
- net 12v: now also R45.1
- net 5v: now also R46.1
- net GND1: now also C22.2, D15.1 (K), D16.1 (K)
- new net: D15.2 (A), R45.2
- new net: D16.2 (A), R46.2
Other:
- note added: "Choose one of the two"
- moved on the sheet: D14, F2, F3, J19, R44, SW2

Commit message: ya
Parts:
- removed J1, J20: Conn_01x05, symbol Connector_Generic:Conn_01x05
- added C23: C, symbol Device:C
- added J1, J22: Conn_01x03_MountingPin, symbol Connector_Generic_MountingPin:Conn_01x03_MountingPin
- added J21: Conn_01x02_Pin, symbol Connector:Conn_01x02_Pin
Connections:
- net GND is gone; now on net GND1: C14.2, C15.2, C16.2, C18.2, C19.2, C20.2, C21.2, J15.2 (Pin_2), J18.N (NEG), Q2.2 (S), R29.2, U1.2 (VSS), U1.5 (VSS), U3.4 (GND), U3.5 (RTH), U3.6 (WDI)
- net +12V: now also U2.48 (VIN), C23.1
- net 44.4V: now also J21.2 (Pin_2)
- net Direction MD1: now also J22.1 (Pin_1)
- net Direction MD2: now also J1.1 (Pin_1)
- net Distance Sensor 5 12V: now also U2.16 (24_A10_TX6_SCL2); no longer U2.15 (3V3)
- net Distance Sensor 6 12V: now also U2.17 (25_A11_RX6_SDA2); no longer U2.16 (24_A10_TX6_SCL2)
- net Distance Sensor 7 12V: now also U2.18 (26_A12_MOSI1); no longer U2.17 (25_A11_RX6_SDA2)
- net Distance Sensor 8 12V: now also U2.19 (27_A13_SCK1); no longer U2.18 (26_A12_MOSI1)
- net Distance Sensor 9 12V: now also U2.20 (28_RX7); no longer U2.19 (27_A13_SCK1)
- net GND1: now also U2.1 (GND), U2.47 (GND), C23.2, J1.3 (Pin_3), J21.1 (Pin_1), J22.3 (Pin_3)
- net PWM MD1: now also J22.2 (Pin_2)
- net PWM MD2: now also J1.2 (Pin_2)
- no-connect marks 5 -> 48
Other:
- note added: "18 Ohm"
- note added: "88 ohm"
- note added: "XT60 to motors"
- note removed: "This 5V is an input Not sure if needed"

Commit message: adding footprints
Parts:
- removed C18, C19, C20, C21: 100nF, symbol Device:C_Small
- removed C23: C, symbol Device:C
- removed D14: LED, symbol Device:LED
- removed F2, F3: Fuse, symbol Device:Fuse
- removed J14: Conn_01x03_MountingPin, symbol Connector_Generic_MountingPin:Conn_01x03_MountingPin
- removed J19: Battery Connector, symbol Connector:Conn_01x02_Socket
- removed R44: 2k Ohm, symbol Device:R_Small_US
- removed R45: R, symbol Device:R
- removed SW2: SW_DIP_x01, symbol Switch:SW_DIP_x01
- added C18, C19, C20, C21, C24: C, Capacitor_SMD:C_0603_1608Metric_Pad1.08x0.95mm_HandSolder, symbol Device:C
- added J19: Conn_01x03_MountingPin, Jst Xh 2.5-3 Pin:JST_B3B-XH-A_LF__SN_, symbol Connector_Generic_MountingPin:Conn_01x03_MountingPin
- added R44: R, Resistor_SMD:R_0603_1608Metric_Pad0.98x0.95mm_HandSolder, symbol Device:R
- C1, C10, C11, C12, C13, C14, C2, C22, C3, C4, C5, C6, C7, C8, C9: footprint (none) -> Capacitor_SMD:C_0603_1608Metric_Pad1.08x0.95mm_HandSolder
- J1, J10, J11, J12, J13, J2, J22, J3, J4, J5, J6, J7, J8, J9: footprint (none) -> Jst Xh 2.5-3 Pin:JST_B3B-XH-A_LF__SN_
- R1, R10, R11, R12, R13, R14, R15, R16, R17, R18, R19, R2, R20, R21, R22, R23, R24, R25, R26, R3, R31, R32, R33, R34, R35, R36, R37, R38, R39, R4, R40, R41, R42, R43, R5, R6, R7, R8, R9: footprint (none) -> Resistor_SMD:R_0603_1608Metric_Pad0.98x0.95mm_HandSolder
- R46: footprint (none) -> Resistor_SMD:R_1206_3216Metric_Pad1.30x1.75mm_HandSolder
Connections:
- net +12V: no longer C1.1, C13.1, C2.1, C22.1, C3.1, J16.1 (Pin_1), J2.2 (Pin_2), J3.2 (Pin_2), J4.2 (Pin_2), U2.48 (VIN)
- net +3.3V: now also C14.2, U2.46 (3V3); no longer C14.1
- net 12v: now also C19.1, R44.1; no longer U1.3 (ON/OFF)
- net 44.4v: now also C18.1, C20.1
- net 5v: now also C21.1
- net Direction MD1: now also U2.3 (1_TX1_CTX2_MISO1)
- net Distance Sensor 1 12V: now also J5.1 (Pin_1); no longer J6.1 (Pin_1)
- net Distance Sensor 2 12V: now also J6.1 (Pin_1); no longer J7.1 (Pin_1)
- net Distance Sensor 3 12V: now also J7.1 (Pin_1); no longer J8.1 (Pin_1)
- net Distance Sensor 4 12V: now also J8.1 (Pin_1); no longer J9.1 (Pin_1)
- net Distance Sensor 5 12V: now also J9.1 (Pin_1); no longer J10.1 (Pin_1)
- net Distance Sensor 6 12V: now also J10.1 (Pin_1); no longer J11.1 (Pin_1)
- net Distance Sensor 7 12V: now also J11.1 (Pin_1); no longer J12.1 (Pin_1)
- net Distance Sensor 8 12V: now also J12.1 (Pin_1); no longer J13.1 (Pin_1)
- net Distance Sensor 9 12V: now also J13.1 (Pin_1)
- net GND1: now also C14.1, U1.3 (ON/OFF), C18.2, C19.2, C20.2, C21.2, C24.2, J19.3 (Pin_3); no longer C14.2
- net Line Sensor 1 5v: now also J19.1 (Pin_1); no longer J2.1 (Pin_1)
- net Line Sensor 2 5v: now also J2.1 (Pin_1); no longer J3.1 (Pin_1)
- net Line Sensor 3 5v: now also J3.1 (Pin_1); no longer J4.1 (Pin_1)
- net Line Sensor 4 5v: now also J4.1 (Pin_1); no longer J5.1 (Pin_1)
- net PWM MD1: now also U2.4 (2_OUT2)
- net at D15.2 (A): now also R44.2
- new net +5V: C1.1, C13.1, C2.1, C22.1, C24.1, C3.1, J16.1 (Pin_1), J19.2 (Pin_2), J2.2 (Pin_2), J3.2 (Pin_2), J4.2 (Pin_2), U2.48 (VIN)
- no-connect marks 48 -> 62
Other:
- note added: "LEDs for 12V and 5V"
- note removed: "Choose one of the two"
- note removed: "Physically split through cable"
- note removed: "motor driver"
- note removed: "sensors"
- note removed: "teensi"
- note removed: "voltage regulator"
- moved on the sheet: C15, C16, C17, F1, J17, J18, J22, Q1, Q2, R27, R28, R29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
